Commit message: 2026 10.3-LLM-control重构优化

File: src/camera_ws/realsense2_gz_description/urdf/_d435.gazebo.xacro (robot description, xacro)
@@ -99,4 +99,5 @@
   depth_near_m:=0.28
   depth_far_m:=3.0
+  native_depth_enabled:=true
   triggered:=false">
     <!-- Realsense D435 RGB properties
@@ -138,15 +139,17 @@
                                            max_depth="${depth_far_m}"
                                            camera_info_topic="${gz_topic_name}/aligned_depth/camera_info"/>
-        <xacro:gazebo_depth_camera name="${name}"
-                                   fps="${fps}"
-                                   gz_topic_name="${gz_topic_name}/native_depth/image"
-                                   image_width="${depth_image_width}"
-                                   image_height="${depth_image_height}"
-                                   fx="${depth_fx}" fy="${depth_fy}" cx="${depth_cx}" cy="${depth_cy}"
-                                   k1="${depth_k1}" k2="${depth_k2}" k3="${depth_k3}" p1="${depth_p1}" p2="${depth_p2}"
-                                   h_fov="${depth_h_fov}"
-                                   v_fov="${depth_v_fov}"
-                                   min_depth="${depth_near_m}"
-                                   max_depth="${depth_far_m}"/>
+        <xacro:if value="${native_depth_enabled}">
+            <xacro:gazebo_depth_camera name="${name}"
+                                       fps="${fps}"
+                                       gz_topic_name="${gz_topic_name}/native_depth/image"
+                                       image_width="${depth_image_width}"
+                                       image_height="${depth_image_height}"
+                                       fx="${depth_fx}" fy="${depth_fy}" cx="${depth_cx}" cy="${depth_cy}"
+                                       k1="${depth_k1}" k2="${depth_k2}" k3="${depth_k3}" p1="${depth_p1}" p2="${depth_p2}"
+                                       h_fov="${depth_h_fov}"
+                                       v_fov="${depth_v_fov}"
+                                       min_depth="${depth_near_m}"
+                                       max_depth="${depth_far_m}"/>
+        </xacro:if>
     </xacro:if>
 </xacro:macro>

File: src/myrobot_simulation/config/robots/fairino3_v6/fairino3_v6_sim.urdf.xacro (robot description, xacro)
@@ -23,4 +23,5 @@
   <xacro:arg name="camera_depth_near_m" default="0.28"/>
   <xacro:arg name="camera_depth_far_m" default="3.0"/>
+  <xacro:arg name="native_depth_enabled" default="true"/>
   <xacro:include filename="$(find fairino_description)/urdf/fairino3_v6.urdf"/>
   <xacro:include filename="$(find fairino_arm_moveit_descriptions)/urdf/camera/camera.xacro"/>
@@ -41,5 +42,6 @@
       depth_k1="$(arg camera_depth_k1)" depth_k2="$(arg camera_depth_k2)" depth_k3="$(arg camera_depth_k3)" depth_p1="$(arg camera_depth_p1)" depth_p2="$(arg camera_depth_p2)"
       depth_h_fov="$(arg camera_depth_h_fov)" depth_v_fov="$(arg camera_depth_v_fov)"
-      depth_near_m="$(arg camera_depth_near_m)" depth_far_m="$(arg camera_depth_far_m)"/>
+      depth_near_m="$(arg camera_depth_near_m)" depth_far_m="$(arg camera_depth_far_m)"
+      native_depth_enabled="$(arg native_depth_enabled)"/>
   </xacro:if>
   <xacro:gz_six_axis_velocity_control

File: src/myrobot_simulation/config/robots/fairino_arm/fairino_arm_inhand_sim.urdf.xacro (robot description, xacro)
@@ -23,4 +23,5 @@
   <xacro:arg name="camera_depth_near_m" default="0.28"/>
   <xacro:arg name="camera_depth_far_m" default="3.0"/>
+  <xacro:arg name="native_depth_enabled" default="true"/>
   <xacro:include filename="$(find fairino_arm_moveit_descriptions)/urdf/fairino_arm_moveit_descriptions.urdf"/>
   <xacro:include filename="$(find fairino_arm_moveit_descriptions)/urdf/camera/camera.xacro"/>
@@ -28,5 +29,5 @@
   <xacro:include filename="../common/sim_plugins.xacro"/>
   <xacro:include filename="../common/sim_ros2_control.xacro"/>
-  <xacro:macro name="fairino_arm_gazebo_handeye_camera" params="camera_fps:=30 camera_image_width:=1280 camera_image_height:=720 camera_fx:=0 camera_fy:=0 camera_cx:=0 camera_cy:=0 camera_k1:=0 camera_k2:=0 camera_k3:=0 camera_p1:=0 camera_p2:=0 camera_noise_stddev:=0 camera_h_fov:=1.2042771838760873 camera_v_fov:=0.7330382858376184 camera_depth_image_width:=1280 camera_depth_image_height:=720 camera_depth_fx:=0 camera_depth_fy:=0 camera_depth_cx:=0 camera_depth_cy:=0 camera_depth_k1:=0 camera_depth_k2:=0 camera_depth_k3:=0 camera_depth_p1:=0 camera_depth_p2:=0 camera_depth_h_fov:=1.5184364492350666 camera_depth_v_fov:=1.0122909661567112 camera_depth_near_m:=0.28 camera_depth_far_m:=3.0">
+  <xacro:macro name="fairino_arm_gazebo_handeye_camera" params="camera_fps:=30 camera_image_width:=1280 camera_image_height:=720 camera_fx:=0 camera_fy:=0 camera_cx:=0 camera_cy:=0 camera_k1:=0 camera_k2:=0 camera_k3:=0 camera_p1:=0 camera_p2:=0 camera_noise_stddev:=0 camera_h_fov:=1.2042771838760873 camera_v_fov:=0.7330382858376184 camera_depth_image_width:=1280 camera_depth_image_height:=720 camera_depth_fx:=0 camera_depth_fy:=0 camera_depth_cx:=0 camera_depth_cy:=0 camera_depth_k1:=0 camera_depth_k2:=0 camera_depth_k3:=0 camera_depth_p1:=0 camera_depth_p2:=0 camera_depth_h_fov:=1.5184364492350666 camera_depth_v_fov:=1.0122909661567112 camera_depth_near_m:=0.28 camera_depth_far_m:=3.0 native_depth_enabled:=true">
     <xacro:camera_v0 parent="tool0">
       <origin xyz="0.000 -0.05 -0.09" rpy="0 -1.57079632679 -1.57079632679"/>
@@ -41,5 +42,6 @@
       depth_k1="${camera_depth_k1}" depth_k2="${camera_depth_k2}" depth_k3="${camera_depth_k3}" depth_p1="${camera_depth_p1}" depth_p2="${camera_depth_p2}"
       depth_h_fov="${camera_depth_h_fov}" depth_v_fov="${camera_depth_v_fov}"
-      depth_near_m="${camera_depth_near_m}" depth_far_m="${camera_depth_far_m}"/>
+      depth_near_m="${camera_depth_near_m}" depth_far_m="${camera_depth_far_m}"
+      native_depth_enabled="${native_depth_enabled}"/>
   </xacro:macro>
   <xacro:gz_common_plugins controllers_file="$(arg controllers_file)" enable_sensors="$(arg enable_camera)"/>
@@ -58,5 +60,6 @@
       camera_depth_k1="$(arg camera_depth_k1)" camera_depth_k2="$(arg camera_depth_k2)" camera_depth_k3="$(arg camera_depth_k3)" camera_depth_p1="$(arg camera_depth_p1)" camera_depth_p2="$(arg camera_depth_p2)"
       camera_depth_h_fov="$(arg camera_depth_h_fov)" camera_depth_v_fov="$(arg camera_depth_v_fov)"
-      camera_depth_near_m="$(arg camera_depth_near_m)" camera_depth_far_m="$(arg camera_depth_far_m)"/>
+      camera_depth_near_m="$(arg camera_depth_near_m)" camera_depth_far_m="$(arg camera_depth_far_m)"
+      native_depth_enabled="$(arg native_depth_enabled)"/>
   </xacro:if>
   <xacro:gz_link_friction link="finger1" mu1="500.0" mu2="500.0" kp="30000" kd="15"/>

File: src/myrobot_simulation/config/robots/fairino_arm/fairino_arm_onbase_sim.urdf.xacro (robot description, xacro)
@@ -23,4 +23,5 @@
   <xacro:arg name="camera_depth_near_m" default="0.28"/>
   <xacro:arg name="camera_depth_far_m" default="3.0"/>
+  <xacro:arg name="native_depth_enabled" default="true"/>
   <xacro:include filename="$(find fairino_arm_moveit_descriptions)/urdf/fairino_arm_moveit_descriptions.urdf"/>
   <xacro:include filename="$(find fairino_arm_moveit_descriptions)/urdf/camera/camera.xacro"/>
@@ -28,5 +29,5 @@
   <xacro:include filename="../common/sim_plugins.xacro"/>
   <xacro:include filename="../common/sim_ros2_control.xacro"/>
-  <xacro:macro name="fairino_arm_gazebo_camera" params="camera_fps:=60 camera_image_width:=640 camera_image_height:=480 camera_fx:=0 camera_fy:=0 camera_cx:=0 camera_cy:=0 camera_k1:=0 camera_k2:=0 camera_k3:=0 camera_p1:=0 camera_p2:=0 camera_noise_stddev:=0 camera_h_fov:=1.2042771838760873 camera_v_fov:=0.7330382858376184 camera_depth_image_width:=1280 camera_depth_image_height:=720 camera_depth_fx:=0 camera_depth_fy:=0 camera_depth_cx:=0 camera_depth_cy:=0 camera_depth_k1:=0 camera_depth_k2:=0 camera_depth_k3:=0 camera_depth_p1:=0 camera_depth_p2:=0 camera_depth_h_fov:=1.5184364492350666 camera_depth_v_fov:=1.0122909661567112 camera_depth_near_m:=0.28 camera_depth_far_m:=3.0">
+  <xacro:macro name="fairino_arm_gazebo_camera" params="camera_fps:=60 camera_image_width:=640 camera_image_height:=480 camera_fx:=0 camera_fy:=0 camera_cx:=0 camera_cy:=0 camera_k1:=0 camera_k2:=0 camera_k3:=0 camera_p1:=0 camera_p2:=0 camera_noise_stddev:=0 camera_h_fov:=1.2042771838760873 camera_v_fov:=0.7330382858376184 camera_depth_image_width:=1280 camera_depth_image_height:=720 camera_depth_fx:=0 camera_depth_fy:=0 camera_depth_cx:=0 camera_depth_cy:=0 camera_depth_k1:=0 camera_depth_k2:=0 camera_depth_k3:=0 camera_depth_p1:=0 camera_depth_p2:=0 camera_depth_h_fov:=1.5184364492350666 camera_depth_v_fov:=1.0122909661567112 camera_depth_near_m:=0.28 camera_depth_far_m:=3.0 native_depth_enabled:=true">
     <xacro:property name="PI" value="3.14159274"/>
     <xacro:camera_v0 parent="base_link">
@@ -42,5 +43,6 @@
       depth_k1="${camera_depth_k1}" depth_k2="${camera_depth_k2}" depth_k3="${camera_depth_k3}" depth_p1="${camera_depth_p1}" depth_p2="${camera_depth_p2}"
       depth_h_fov="${camera_depth_h_fov}" depth_v_fov="${camera_depth_v_fov}"
-      depth_near_m="${camera_depth_near_m}" depth_far_m="${camera_depth_far_m}"/>
+      depth_near_m="${camera_depth_near_m}" depth_far_m="${camera_depth_far_m}"
+      native_depth_enabled="${native_depth_enabled}"/>
   </xacro:macro>
   <xacro:gz_common_plugins controllers_file="$(arg controllers_file)" enable_sensors="$(arg enable_camera)"/>
@@ -59,5 +61,6 @@
       camera_depth_k1="$(arg camera_depth_k1)" camera_depth_k2="$(arg camera_depth_k2)" camera_depth_k3="$(arg camera_depth_k3)" camera_depth_p1="$(arg camera_depth_p1)" camera_depth_p2="$(arg camera_depth_p2)"
       camera_depth_h_fov="$(arg camera_depth_h_fov)" camera_depth_v_fov="$(arg camera_depth_v_fov)"
-      camera_depth_near_m="$(arg camera_depth_near_m)" camera_depth_far_m="$(arg camera_depth_far_m)"/>
+      camera_depth_near_m="$(arg camera_depth_near_m)" camera_depth_far_m="$(arg camera_depth_far_m)"
+      native_depth_enabled="$(arg native_depth_enabled)"/>
   </xacro:if>
   <xacro:gz_link_friction link="finger1" mu1="500.0" mu2="500.0" kp="30000" kd="15"/>

File: src/myrobot_support_ws/fairino_arm_moveit_descriptions/urdf/camera/camera.xacro (robot description, xacro)
@@ -44,5 +44,5 @@
 	</xacro:macro>
 	<!-- =========================================================宏 2：Gazebo 中的相机传感器 / 材质========================================================= -->
-	<xacro:macro name="camera_gazebo_v0" params="sensor_type:=rgbd fps:=60 image_width:=640 image_height:=480 fx:=0 fy:=0 cx:=0 cy:=0 k1:=0 k2:=0 k3:=0 p1:=0 p2:=0 noise_stddev:=0 h_fov:=1.2042771838760873 v_fov:=0.7330382858376184 depth_image_width:=1280 depth_image_height:=720 depth_fx:=0 depth_fy:=0 depth_cx:=0 depth_cy:=0 depth_k1:=0 depth_k2:=0 depth_k3:=0 depth_p1:=0 depth_p2:=0 depth_h_fov:=1.5184364492350666 depth_v_fov:=1.0122909661567112 depth_near_m:=0.28 depth_far_m:=3.0">
+	<xacro:macro name="camera_gazebo_v0" params="sensor_type:=rgbd fps:=60 image_width:=640 image_height:=480 fx:=0 fy:=0 cx:=0 cy:=0 k1:=0 k2:=0 k3:=0 p1:=0 p2:=0 noise_stddev:=0 h_fov:=1.2042771838760873 v_fov:=0.7330382858376184 depth_image_width:=1280 depth_image_height:=720 depth_fx:=0 depth_fy:=0 depth_cx:=0 depth_cy:=0 depth_k1:=0 depth_k2:=0 depth_k3:=0 depth_p1:=0 depth_p2:=0 depth_h_fov:=1.5184364492350666 depth_v_fov:=1.0122909661567112 depth_near_m:=0.28 depth_far_m:=3.0 native_depth_enabled:=true">
         <!-- Gazebo 侧 D435 相机 -->
         <xacro:gazebo_d435
@@ -62,5 +62,6 @@
             depth_k1="${depth_k1}" depth_k2="${depth_k2}" depth_k3="${depth_k3}" depth_p1="${depth_p1}" depth_p2="${depth_p2}"
             depth_h_fov="${depth_h_fov}" depth_v_fov="${depth_v_fov}"
-            depth_near_m="${depth_near_m}" depth_far_m="${depth_far_m}"/>
+            depth_near_m="${depth_near_m}" depth_far_m="${depth_far_m}"
+            native_depth_enabled="${native_depth_enabled}"/>
         <!-- camera_link 材质：使用 URDF visual 自带的材质，不强制覆盖 -->
     </xacro:macro>
